File: urine_dipstick_analyzer.kicad_sch (KiCad schematic)
At the start: 46 parts, among them Q1 2N7000, Q2 IRLZ44N, Q3 IRLZ44N, Q4 2N7000, SW1 Measure, SW2 Limit, SW3 Reed_Switch

Commit message: Fix schematic pin overlaps and add BOM/render tools
- Widen ESP32 block to 76.20mm, all modules to 38-43mm
- Increase pin spacing to 7.62mm with wire stubs for label clearance
- Adjust section coordinates to prevent block collisions
- Add BOM CSV/PDF generator with 72-part costed bill of materials
- Add matplotlib schematic renderer for PNG preview

Co-Authored-By: Claude Opus 4.6 <noreply@anthropic.com>
Parts:
- removed D5: Red, symbol Device:LED
- removed D6: Green, symbol Device:LED
- removed D7: Blue, symbol Device:LED
- removed Q4: 2N7000, symbol Device:Q_NMOS_GDS
- removed R15, R16, R17: 330, symbol Device:R
- removed R18: 10k, symbol Device:R
- added C15, C16, C17, C19: 100nF, symbol Device:C
- added C18: 100uF, symbol Device:C
- C11: value 10uF -> 100nF
- C13: value 100uF -> 10uF
- C3, C8: value 100nF -> 10uF
- D1: value White -> UV-C
- D2: value White -> Red
- D3: value White -> Green
- D4: value UV-C -> Blue
- Q1: value 2N7000 -> IRLZ44N
- Q3: value IRLZ44N -> 2N7000
- R10: value 47 -> 10k
- R11, R12, R13: value 10k -> 330R
- R6, R8: value 330 -> 10k
- R7: value 330 -> 47R
- SW3: value Reed_Switch -> MC-38_Reed
Connections:
- net 3V3: now also Q1.3 (S), Q2.3 (S), Q3.3 (S), SW1.1, SW2.1, SW3.1
- net 5V: now also Q3.2 (D)
- net 9V: now also Q2.2 (D)
- net FAN_GATE: now also Q3.1 (G)
- net HEATER_GATE: now also Q2.1 (G)
- net LIMIT_SW: now also SW2.2
- net MEASURE_BTN: now also SW1.2
- net REED_SW: now also SW3.2
- net UV_GATE: now also Q1.1 (G)
- net UV_DRAIN: now reaches Q1.2 (D)
Other:
- note added: "(+) GPIO21"
- note added: "32K"
- note added: "ADDR"
- note added: "ALT"
- note added: "BARCODE_RX"
- note added: "BARCODE_TX"
- note added: "BT1: LiPo 3.7V 2000mAh"
- note added: "CAMERA & OPTICS"
- note added: "CELL"
- note added: "D0"
- note added: "D1"
- note added: "D2"
- note added: "D3"
- note added: "D4"
- note added: "D5"
- note added: "D6"
- note added: "D7"
- note added: "DC"
- note added: "DISPLAY & STORAGE"
- note added: "EN"
- note added: "ESP32-S3 MCU"
- note added: "GPIO10"
- note added: "GPIO11"
- note added: "GPIO12"
- note added: "GPIO13"
- note added: "GPIO14"
- note added: "GPIO35"
- note added: "GPIO36"
- note added: "GPIO37"
- note added: "GPIO45"
- note added: "GPIO46"
- note added: "GPIO47"
- note added: "GPIO48"
- note added: "GPIO9"
- note added: "LED"
- note added: "MC-38 Reed Switch Interlock"
- note added: "MOTOR & ACTUATORS"
- note added: "MS1"
- note added: "MS2"
- note added: "NTC Thermistor Divider"
- note added: "POWER SUPPLY"
- note added: "PROG"
- note added: "RGB Status LED (Common Anode)"
- note added: "RST"
- note added: "SAFETY"
- note added: "SENSORS & I2C"
- note added: "SIOC"
- note added: "SIOD"
- note added: "SPI_MISO"
- note added: "SQW"
- note added: "STAT1"
- note added: "STAT2"
- note added: "TRIG"
- note added: "U10: ILI9341 2.4in TFT"
- note added: "U11: SD Card Module (SPI)"
- note added: "U12: A4988 Stepper Driver"
- note added: "U13: GM65 Barcode Scanner"
- note added: "U2: Pololu S13V25F9 (9V)"
- note added: "U3: Pololu S7V8F3 (3.3V)"
- note added: "U4: MAX17048 Fuel Gauge"
- note added: "U6: SHT31 Humidity Sensor"
- note added: "U7: BH1750 Light Sensor"
- note added: "U8: DS3231 RTC"
- note added: "U9: OV2640 Camera"
- note added: "UI: BUTTON / LED / BUZZER"
- note added: "VBAT"
- note added: "VIN"
- note added: "VIN (USB-C)"
- note added: "VOUT (3.3V)"
- note added: "VOUT (9V)"
- note added: "VSS"
- note removed: "(common anode through resistors)"
- note removed: "3.3V Distributed"
- note removed: "3.3V Rail"
- note removed: "3.7V LiPo"
- note removed: "5V Rail"
- note removed: "9V Distributed"
- note removed: "9V Rail"
- note removed: "=== CAMERA & OPTICS ==="
- note removed: "=== ESP32-S3 MCU ==="
- note removed: "=== MOTOR & ACTUATORS ==="
- note removed: "=== POWER NETS ==="
- note removed: "=== POWER SUPPLY ==="
- note removed: "=== SAFETY ==="
- note removed: "=== SENSORS & I2C ==="
- note removed: "=== USER INTERFACE ==="
- note removed: "BT1: LiPo 3.7V 1000mAh"
- note removed: "Buck-Boost 5V/9V"
- note removed: "Buzzer Circuit"
- note removed: "D0-D7"
- note removed: "DVP_D0-D7"
- note removed: "DVP_HREF"
- note removed: "DVP_PCLK"
- note removed: "DVP_VSYNC"
- note removed: "DVP_XCLK"
- note removed: "Ground Distributed"
- note removed: "MCU Buck-Boost 3.3V"
- note removed: "RGB Status LED"
- note removed: "Reed Switch Safety Interlock"
- note removed: "Thermistor Circuit"
- note removed: "U10: OV2640 Camera + CPL Filter"
- note removed: "U11: A4988 Stepper Driver"
- note removed: "U12: SD Card Module (SPI)"
- note removed: "U2: Pololu S13V25F9"
- note removed: "U3: Pololu S7V8F3"
- note removed: "U4: Power Management PCB"
- note removed: "U6: OLED Display (SSD1306)"
- note removed: "U7: SHT31 Humidity Sensor"
- note removed: "U8: BH1750 Light Sensor"
- note removed: "U9: Barcode Scanner (UART)"
- note removed: "White LED Array"
- title: Urine Dipstick Analyzer -> Urine Dipstick Analyzer v2.0

Commit message: Add professional section boxes and fix schematic layout
- Dashed boundary rectangles around each section (like reference schematic)
- Layout instructions text block at bottom
- Fixed section spacing to prevent overlap between Motor/UI and Display/Safety
- ESP32 pins fully readable with 7.62mm spacing and 76.20mm box width

Co-Authored-By: Claude Opus 4.6 <noreply@anthropic.com>
Other:
- note added: "1. All decoupling caps should be placed as close to IC VCC pins as possible."
- note added: "2. I2C bus pull-ups: single pair of 4.7k at MCU end."
- note added: "3. SPI bus shared between TFT display and SD card (active-low CS per device)."
- note added: "4. All MOSFETs are low-side switches with 10k gate pull-downs."
- note added: "5. UV-C LED requires series current-limiting resistor (47R @ 9V)."
- note added: "Camera & Optics Section"
- note added: "Display & Storage Section"
- note added: "Layout Instructions:"
- note added: "MCU & GPIO Section"
- note added: "Motor & Actuator Section"
- note added: "Power Supply Section"
- note added: "Safety Section"
- note added: "Sensors & I2C Section"
- note added: "UI: Button / LED / Buzzer Section"
- note removed: "POWER SUPPLY"

Commit message: Fix KiCad schematic: proper IC symbols with wired connections
- Complete rewrite of generate_schematic.py with real lib_symbols
- All ICs now have proper pin definitions (not just wire rectangles)
- Decoupling caps explicitly wired to IC VDD/GND pins
- Fan (FAN1) added as 2-terminal component wired to Q3 drain + 5V
- OV2640 camera data bus (D0-D7) connected to ESP32 via net labels
- Fixed KiCad 10 subsymbol naming (no library prefix in sub-symbol names)
- Stripped non-ASCII characters for KiCad parser compatibility
- 57 symbol instances, 71 wires, 93 net labels, 94 global labels

Co-Authored-By: Claude Opus 4.6 <noreply@anthropic.com>
Parts:
- removed C1, C10, C11, C12, C14, C15, C16, C17, C19, C2, C4, C6, C7, C9: 100nF, symbol Device:C
- removed C13, C3, C5, C8: 10uF, symbol Device:C
- removed C18: 100uF, symbol Device:C
- removed D1: UV-C, symbol Device:LED
- removed D2: Red, symbol Device:LED
- removed D3: Green, symbol Device:LED
- removed D4: Blue, symbol Device:LED
- removed Q1, Q2: IRLZ44N, symbol Device:Q_NMOS_GDS
- removed Q3: 2N7000, symbol Device:Q_NMOS_GDS
- removed R1, R2: 4.7k, symbol Device:R
- removed R10, R14, R4, R5, R6, R8, R9: 10k, symbol Device:R
- removed R11, R12, R13: 330R, symbol Device:R
- removed R3: NTC 10k, symbol Device:R
- removed R7: 47R, symbol Device:R
- removed SW1: Measure, symbol Switch:SW_Push
- removed SW2: Limit, symbol Switch:SW_Push
- removed SW3: MC-38_Reed, symbol Switch:SW_Push
- added C1: 4.7uF, symbol custom:C
- added C10, C11, C12, C14, C15, C16, C19, C2, C4, C6, C7, C9: 100nF, symbol custom:C
- added C13, C3, C5, C8: 10uF, symbol custom:C
- added C17: 100uF, symbol custom:C
- added D1: UV-C LED, symbol custom:LED
- added D2: Red LED, symbol custom:LED
- added D3: Green LED, symbol custom:LED
- added D4: Blue LED, symbol custom:LED
- added FAN1: Fan, symbol custom:FAN
- added M1: NEMA-17, symbol custom:NEMA17
- added Q1, Q2: IRLZ44N, symbol custom:NMOSFET
- added R1, R2: 4.7k, symbol custom:R
- added R10, R14, R4, R5, R6, R8, R9, R_PROG: 10k, symbol custom:R
- added R11, R12, R13: 330R, symbol custom:R
- added R3: NTC 10k, symbol custom:R
- added R7: 47R, symbol custom:R
- added SW1: Measure, symbol custom:SW_Push
- added SW2: Limit, symbol custom:SW_Push
- added SW3: MC-38 Reed, symbol custom:SW_Push
- added U1: MCP73833, symbol custom:MCP73833
- added U10: ILI9341, symbol custom:ILI9341
- added U11: SD Card Module, symbol custom:GM65
- added U12: A4988, symbol custom:A4988
- added U13: GM65 Barcode, symbol custom:GM65
- added U2: S13V25F9 (9V), symbol custom:REG9V
- added U3: S7V8F3 (3.3V), symbol custom:REG3V3
- added U4: MAX17048, symbol custom:MAX17048
- added U5: ESP32-S3-WROOM-1, symbol custom:ESP32S3
- added U6: SHT31, symbol custom:SHT31
- added U7: BH1750, symbol custom:BH1750
- added U8: DS3231, symbol custom:DS3231
- added U9: OV2640, symbol custom:OV2640
Connections:
- net 3V3: now also D2.2 (K), D3.2 (K), D4.2 (K), U10.3 (CS), U11.1 (VCC), U13.1 (VCC), U3.3 (VOUT), U5.2 (IO0), U9.7 (SIOD), U9.9 (VSYNC)
- net 5V: now also FAN1.1 (+)
- net 9V: now also D1.1 (A), Q2.3 (S), U2.3 (VOUT)
- net BARCODE_RX: now also U13.3 (TX), U5.37 (IO47)
- net BARCODE_TX: now also U5.38 (IO48)
- net BUZZER: now also U5.40 (TX)
- net CAM_D0: now also U5.36 (IO46), U9.18 (PCLK)
- net CAM_D1: now also U5.35 (IO45), U9.17 (D7)
- net CAM_D2: now also U5.34 (IO44), U9.16 (D6)
- net CAM_D3: now also U5.33 (IO43), U9.15 (D5)
- net CAM_D4: now also U5.32 (IO42), U9.14 (D4)
- net CAM_D5: now also U5.31 (IO41), U9.13 (D3)
- net CAM_D6: now also U5.30 (IO40), U9.12 (D2)
- net CAM_D7: now also U5.29 (IO39), U9.11 (D1)
- net CAM_HREF: now also U5.26 (IO36), U9.2 (GND)
- net CAM_PCLK: now also U5.28 (IO38), U9.10 (D0)
- net CAM_SIOD: now also U5.24 (IO21), U9.3 (RESETB)
- net CAM_VSYNC: now also U5.27 (IO37), U9.1 (VDD3V3)
- net CAM_XCLK: now also U5.25 (IO35), U9.5 (XCLK)
- net DIR: now also U5.6 (IO4)
- net FAN_GATE: now also U5.19 (IO19)
- net HEATER_GATE: now also Q2.1 (G), U5.7 (IO5)
- net I2C_SCL: now also U5.4 (IO2), U9.4 (PWDN)
- net I2C_SDA: now also U5.3 (IO1)
- net LIMIT_SW: now also SW2.2, U5.5 (IO3)
- net MEASURE_BTN: now also SW1.2, U5.20 (3V3)
- net REED_SW: now also SW3.2
- net RGB_B: now also U5.14 (IO12)
- net RGB_G: now also U5.15 (IO13)
- net RGB_R: now also U5.16 (IO14)
- net SD_CS: now also U11.3 (TX), U5.39 (GND)
- net SPI_MISO: now also U10.6 (MISO), U5.22 (IO17)
- net SPI_MOSI: now also U10.7 (SCK), U5.12 (IO10)
- net SPI_SCK: now also U10.5 (MOSI), U5.11 (IO9)
- net STEP: now also U5.18 (IO18)
- net STEPPER_2A: now also M1.3 (B+)
- net TFT_CS: now also U10.1 (VCC), U5.10 (IO8)
- net TFT_DC: now also U5.9 (IO7)
- net TFT_RST: now also U5.8 (IO6)
- net THERM_ADC: now also U5.13 (IO11)
- net UV_GATE: now also Q1.1 (G), U5.17 (IO15)
- new net GND: Q1.2 (D), Q2.2 (D), SW1.1, SW2.1, SW3.1, U10.2 (GND), U2.1 (VIN), U3.1 (VIN), U5.23 (IO20), U9.6 (SIOC), U9.8 (HREF)
- new net STEPPER_1A: M1.1 (A+)
Other:
- note added: "(+)GPIO21 (-)GND"
- note added: "1 - Power Supply"
- note added: "2 - MCU ESP32-S3"
- note added: "3 - Sensors & I2C"
- note added: "4 - Camera & Optics"
- note added: "5 - Display & SD"
- note added: "6 - Motor & Actuators"
- note added: "7 - UI: Button/LED/Buzzer"
- note added: "8 - Safety"
- note added: "Heater Film (9V)"
- note added: "I2C Pull-ups (4.7k to 3V3)"
- note added: "Layout notes: 1) place decoupling caps next to IC VCC pins. 2) I2C pull-ups at MCU end. 3) SPI shared between TFT & SD (CS per device). 4) All MOSFETs low-side with 10k gate pull-down."
- note removed: "(+) GPIO21"
- note removed: "1. All decoupling caps should be placed as close to IC VCC pins as possible."
- note removed: "1A"
- note removed: "1B"
- note removed: "2. I2C bus pull-ups: single pair of 4.7k at MCU end."
- note removed: "2A"
- note removed: "2B"
- note removed: "3. SPI bus shared between TFT display and SD card (active-low CS per device)."
- note removed: "32K"
- note removed: "3V3"
- note removed: "4. All MOSFETs are low-side switches with 10k gate pull-downs."
- note removed: "5. UV-C LED requires series current-limiting resistor (47R @ 9V)."
- note removed: "A1"
- note removed: "A2"
- note removed: "ADDR"
- note removed: "ALT"
- note removed: "B1"
- note removed: "B2"
- note removed: "BARCODE_RX"
- note removed: "BARCODE_TX"
- note removed: "CAMERA & OPTICS"
- note removed: "CELL"
- note removed: "CS"
- note removed: "Camera & Optics Section"
- note removed: "D0"
- note removed: "D1"
- note removed: "D2"
- note removed: "D3"
- note removed: "D4"
- note removed: "D5"
- note removed: "D6"
- note removed: "D7"
- note removed: "DC"
- note removed: "DIR"
- note removed: "DISPLAY & STORAGE"
- note removed: "Display & Storage Section"
- note removed: "EN"
- note removed: "ESP32-S3 MCU"
- note removed: "GND"
- note removed: "GPIO1"
- note removed: "GPIO10"
- note removed: "GPIO11"
- note removed: "GPIO12"
- note removed: "GPIO13"
- note removed: "GPIO14"
- note removed: "GPIO15"
- note removed: "GPIO16"
- note removed: "GPIO17"
- note removed: "GPIO18"
- note removed: "GPIO19"
- note removed: "GPIO2"
- note removed: "GPIO20"
- note removed: "GPIO21"
- note removed: "GPIO35"
- note removed: "GPIO36"
- note removed: "GPIO37"
- note removed: "GPIO38"
- note removed: "GPIO39"
- note removed: "GPIO4"
- note removed: "GPIO40"
- note removed: "GPIO41"
- note removed: "GPIO42"
- note removed: "GPIO43"
- note removed: "GPIO44"
- note removed: "GPIO45"
- note removed: "GPIO46"
- note removed: "GPIO47"
- note removed: "GPIO48"
- note removed: "GPIO5"
- note removed: "GPIO6"
- note removed: "GPIO7"
- note removed: "GPIO8"
- note removed: "GPIO9"
- note removed: "HREF"
- note removed: "Heater Film"
- note removed: "I2C Pull-ups"
- note removed: "LED"
- note removed: "Layout Instructions:"
- note removed: "Limit Switch"
- note removed: "M1: NEMA 17 Stepper"
- note removed: "MC-38 Reed Switch Interlock"
- note removed: "MCU & GPIO Section"
- note removed: "MISO"
- note removed: "MOSI"
- note removed: "MOTOR & ACTUATORS"
- note removed: "MS1"
- note removed: "MS2"
- note removed: "Measure Button"
- note removed: "Motor & Actuator Section"
- note removed: "PCLK"
- note removed: "PROG"
- note removed: "Power Supply Section"
- note removed: "RST"
- note removed: "RX"
- note removed: "SAFETY"
- note removed: "SCK"
- note removed: "SCL"
- note removed: "SDA"
- note removed: "SENSORS & I2C"
- note removed: "SIOC"
- note removed: "SIOD"
- note removed: "SPI_MISO"
- note removed: "SQW"
- note removed: "STAT1"
- note removed: "STAT2"
- note removed: "STEP"
- note removed: "Safety Section"
- note removed: "Sensors & I2C Section"
- note removed: "TRIG"
- note removed: "TX"
- note removed: "U10: ILI9341 2.4in TFT"
- note removed: "U11: SD Card Module (SPI)"
- note removed: "U12: A4988 Stepper Driver"
- note removed: "U13: GM65 Barcode Scanner"
- note removed: "U1: MCP73833 USB-C Charger"
- note removed: "U2: Pololu S13V25F9 (9V)"
- note removed: "U3: Pololu S7V8F3 (3.3V)"
- note removed: "U4: MAX17048 Fuel Gauge"
- note removed: "U5: ESP32-S3-WROOM-1"
- note removed: "U6: SHT31 Humidity Sensor"
- note removed: "U7: BH1750 Light Sensor"
- note removed: "U8: DS3231 RTC"
- note removed: "U9: OV2640 Camera"
- note removed: "UI: BUTTON / LED / BUZZER"
- note removed: "UI: Button / LED / Buzzer Section"
- note removed: "VBAT"
- note removed: "VCC"
- note removed: "VDD"
- note removed: "VIN"
- note removed: "VIN (USB-C)"
- note removed: "VMOT"
- note removed: "VOUT (3.3V)"
- note removed: "VOUT (9V)"
- note removed: "VSS"
- note removed: "VSYNC"
- note removed: "Vent Fan"
- note removed: "XCLK"
- title: Urine Dipstick Analyzer v2.0 -> Urine Dipstick Analyzer v2.0 - Fixed Wiring
